File: voc_sensor.brd (EAGLE design)
At the start: 28 x 32 mm, 18 parts, among them IC1 MP901, IC2 DS2438, IC4 LMZ21700, X1 SPRING_CLAMP_3_AST215

Commit message: changing D1 and D8 to 12V types, resulting in an increased voltage compared to previous versions of the schematic - but it lowers the expected voltage range, which was 7-17 V - now it is 7-12V related to issue #3
Parts:
- D1, D8: value SMAJ7.5A-LF -> SMAJ12A
Changed lines of the file:
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@@
 <attribute name="VALUE" x="12.795" y="25.065" size="1.016" layer="28" rot="MR90"/>
 </element>
-<element name="D8" library="diodes" package="DO214AC" value="SMAJ7.5A-LF" x="5.7" y="8.9" smashed="yes" rot="MR0">
+<element name="D8" library="diodes" package="DO214AC" value="SMAJ12A" x="5.7" y="8.9" smashed="yes" rot="MR0">
 <attribute name="NAME" x="4.84" y="6.486" size="1" layer="26" font="vector" ratio="20" rot="MR0"/>
 </element>
@@
 <attribute name="VOLTAGE" value="&gt;=25 V" x="17.5" y="27.1" size="1.778" layer="28" rot="MR90" display="off"/>
 </element>
-<element name="D1" library="diodes" package="DO214AC" value="SMAJ7.5A-LF" x="16.4" y="22.8" smashed="yes" rot="MR0">
+<element name="D1" library="diodes" package="DO214AC" value="SMAJ12A" x="16.4" y="22.8" smashed="yes" rot="MR0">
 <attribute name="NAME" x="18.54" y="24.086" size="1" layer="26" font="vector" ratio="20" rot="MR0"/>
 </element>
