File: voc_sensor.sch (EAGLE design)
At the start: 18 parts, among them IC1 MP901, IC2 DS2438, IC4 LMZ21700, X1 SPRING_CLAMP_3_AST215

Commit message: changing D1 and D8 to 12V types, resulting in an increased voltage compared to previous versions of the schematic - but it lowers the expected voltage range, which was 7-17 V - now it is 7-12V related to issue #3
Parts:
- D1, D8: value SMAJ7.5A-LF -> SMAJ12A
Changed lines of the file:
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@@
 <part name="R1" library="rcl" deviceset="R-EU_" device="R0402" value="5.1"/>
 <part name="R2" library="rcl" deviceset="R-EU_" device="R0402" value="5.1"/>
-<part name="D8" library="diodes" deviceset="ZENER" device="" value="SMAJ7.5A-LF"/>
+<part name="D8" library="diodes" deviceset="ZENER" device="" value="SMAJ12A"/>
 <part name="GND1" library="supply1" deviceset="GND" device=""/>
 <part name="GND2" library="supply1" deviceset="GND" device=""/>
@@
 </part>
 <part name="GND3" library="supply1" deviceset="GND" device=""/>
-<part name="D1" library="diodes" deviceset="ZENER" device="" value="SMAJ7.5A-LF"/>
+<part name="D1" library="diodes" deviceset="ZENER" device="" value="SMAJ12A"/>
 <part name="R4" library="rcl" deviceset="R-EU_" device="R0402" value="5.1"/>
 <part name="X1" library="connectors" deviceset="SPRING_CLAMP_3" device="_AST215"/>
